File: hardware/RC-Multiswitch-ESP32-C3.kicad_pcb (KiCad board)
At the start: 2 copper layers, 66.5 x 51.4 mm, 31 parts, among them CN1 UART A, CN2 12V, J1 Ausgaenge, J5 UART B, U1 ESP32-C3 SuperMini, U2 ULN2803A

Commit message: Lokale KiCad-Staende vom 2026-10-17/18 uebernehmen
Die Arbeit lag nur lokal (nicht auf GitHub) und wurde beim Abgleich
nach der Umbenennung ueberschrieben. Wiederhergestellt aus
backups/vor-umbenennung, Dateinamen und Projektverweise auf
RC-Multiswitch angepasst.

Co-Authored-By: Claude Opus 5.5 (1M context) <noreply@anthropic.com>
Claude-Session: https://claude.ai/code/session_01Np9GkYmRMGJmd89YiKPa21
Parts:
- moved J5 7.64 mm to (144.1, 44.9), turned to 180 degrees
Routing:
- net /UB_RX: track 41.5 -> 32.6 mm, vias 1 -> 0
- net /UB_TX: track 38.5 -> 34.3 mm
- net GND: track 143.8 -> 139.8 mm
Other:
- board text added: "UART B RX TX + -"
- board text removed: "UART B TX RX + -"

Commit message: Lastversorgung CN2 auf 5-12 V, Widerstandswerte entfernt
- D1 TVS P6KE33A -> P6KE18A (Schaltplan, PCB, Aufdruck)
- Beschriftung CN2/VLOAD 12-24V -> 5-12V, Aufdruck 5V-24V -> 5V-12V
- R1-R16 ohne Wert: Anwender legt sie selbst aus, LED-Empfehlung steht auf der Platine
- Projektbeschreibung, Hardware-Beschreibung, README angepasst
- ULN2803A und ESP-Versorgung ueber CN1 bleiben unveraendert

Co-Authored-By: Claude Opus 5.5 (1M context) <noreply@anthropic.com>
Claude-Session: https://claude.ai/code/session_015ZTAHN4h1MhX6WfGWCfmx3
Parts:
- CN2: value 12V -> 5-12V
- D1: value P6KE33A -> P6KE18A
- R1, R10, R11, R12, R13, R14, R15, R16, R2, R3, R4, R5, R6, R7, R8, R9: value 150 -> R
Other:
- board text added: "5V-12V"
- board text added: "P6KE18A"
- board text removed: "5V-24V"
- board text removed: "P6KE33A"
Changed lines of the file:
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@@
 			)
 		)
-		(property "Value" "150"
+		(property "Value" "R"
 			(at 3.81 5.3 0)
 			(layer "F.Fab")
@@
 			)
 		)
-		(property "Value" "150"
+		(property "Value" "R"
 			(at 3.81 5.47 0)
 			(layer "F.Fab")
@@
 			)
 		)
-		(property "Value" "P6KE33A"
+		(property "Value" "P6KE18A"
 			(at 6.75 -3.27 180)
 			(layer "F.Fab")
@@
 			)
 		)
-		(property "Value" "150"
+		(property "Value" "R"
 			(at 3.81 2.35 0)
 			(layer "F.Fab")
@@
 			)
 		)
-		(property "Value" "150"
+		(property "Value" "R"
 			(at 3.81 4.05 90)
 			(layer "F.Fab")
@@
 			)
 		)
-		(property "Value" "150"
+		(property "Value" "R"
 			(at 3.81 2.37 0)
 			(layer "F.Fab")
@@
 			)
 		)
-		(property "Value" "150"
+		(property "Value" "R"
 			(at 3.81 2.37 90)
 			(layer "F.Fab")
@@
 			)
 		)
-		(property "Value" "150"
+		(property "Value" "R"
 			(at 3.81 2.37 90)
 			(layer "F.Fab")
@@
 			)
 		)
-		(property "Value" "150"
+		(property "Value" "R"
 			(at 3.81 2.37 90)
 			(layer "F.Fab")
@@
 			)
 		)
-		(property "Value" "150"
+		(property "Value" "R"
 			(at 3.81 2.37 0)
 			(layer "F.Fab")
@@
 			)
 		)
-		(property "Value" "150"
+		(property "Value" "R"
 			(at 3.81 2.37 0)
 			(layer "F.Fab")
@@
 			)
 		)
-		(property "Value" "150"
+		(property "Value" "R"
 			(at 3.81 2.37 90)
 			(layer "F.Fab")
@@
 			)
 		)
-		(property "Value" "150"
+		(property "Value" "R"
 			(at 3.81 2.37 90)
 			(layer "F.Fab")
@@
 			)
 		)
-		(property "Value" "150"
+		(property "Value" "R"
 			(at 3.81 2.37 0)
 			(layer "F.Fab")
@@
 			)
 		)
-		(property "Value" "12V"
+		(property "Value" "5-12V"
 			(at 1 7.45 270)
 			(layer "F.Fab")
@@
 			)
 		)
-		(property "Value" "150"
+		(property "Value" "R"
 			(at 3.81 2.37 90)
 			(layer "F.Fab")
@@
 			)
 		)
-		(property "Value" "150"
+		(property "Value" "R"
 			(at 3.81 2.37 90)
 			(layer "F.Fab")
@@
 			)
 		)
-		(property "Value" "150"
+		(property "Value" "R"
 			(at 3.81 2.37 0)
 			(layer "F.Fab")
@@
 		)
 	)
-	(gr_text "P6KE33A"
+	(gr_text "P6KE18A"
 		(at 139.72 81.9 0)
 		(layer "F.SilkS")
@@
 		)
 	)
-	(gr_text "5V-24V"
+	(gr_text "5V-12V"
 		(at 125.07 80.3 0)
 		(layer "F.SilkS")
