File: hardware/RC-Multiswitch-ESP32-C3.kicad_pcb (KiCad board)
At the start: 2 copper layers, 66.5 x 51.4 mm, 31 parts, among them CN1 UART A, CN2 5-12V, J1 Ausgaenge, J5 UART B, U1 ESP32-C3 SuperMini, U2 ULN2803A

Commit message: PCB: Martins Stand 20.10. (nach Prüfung C3/S3)
Parts:
- added G***: LOGO, LOGO, F.Cu at (129.8, 42.0)
Other:
- board size 66.5 x 51.4 mm -> 66.5 x 50.2 mm
- board text added: "+ -"
