File: hardware/RC-Multiswitch-ESP32-C3.kicad_sch (KiCad schematic)
At the start: 31 parts, among them CN1 UART A, CN2 12V, J1 Ausgaenge, J5 UART B, U1 ESP32-C3 SuperMini, U2 ULN2803A

Commit message: Umbenennung CRSF-Multiswitch -> RC-Multiswitch
Neutraler Name, weil der Multiswitch neben CRSF auch SBUS versteht.
README, docs (MD und DOCX), KiCad-Projekt (Dateinamen, Projekt- und
Sheet-Verweise, Titel), Sketch-Ordner und CI-Pfad angepasst.
Geraetename, WLAN-SSID und Config-Export bleiben "MultiSwitch".

Co-Authored-By: Claude Opus 5.5 (1M context) <noreply@anthropic.com>
Claude-Session: https://claude.ai/code/session_01Np9GkYmRMGJmd89YiKPa21
Other:
- title: CRSF Multiswitch ESP32-C3 SuperMini (ULN2803A) -> RC Multiswitch ESP32-C3 SuperMini (ULN2803A)
Changed lines of the file:
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@@
 	(paper "A4")
 	(title_block
-		(title "CRSF Multiswitch ESP32-C3 SuperMini (ULN2803A)")
+		(title "RC Multiswitch ESP32-C3 SuperMini (ULN2803A)")
 		(date "2026-10-14")
 		(rev "v0.3")
@@
 		)
 		(instances
-			(project "CRSF-Multiswitch-ESP32-C3"
+			(project "RC-Multiswitch-ESP32-C3"
 				(path "/0f0fc713-9c7c-45b9-9629-0d42632ffdae"
 					(reference "LED5")
@@
 		)
 		(instances
-			(project "CRSF-Multiswitch-ESP32-C3"
+			(project "RC-Multiswitch-ESP32-C3"
 				(path "/0f0fc713-9c7c-45b9-9629-0d42632ffdae"
 					(reference "#PWR15")
@@
 		)
 		(instances
-			(project "CRSF-Multiswitch-ESP32-C3"
+			(project "RC-Multiswitch-ESP32-C3"
 				(path "/0f0fc713-9c7c-45b9-9629-0d42632ffdae"
 					(reference "LED4")
@@
 		)
 		(instances
-			(project "CRSF-Multiswitch-ESP32-C3"
+			(project "RC-Multiswitch-ESP32-C3"
 				(path "/0f0fc713-9c7c-45b9-9629-0d42632ffdae"
 					(reference "#FLG06")
@@
 		)
 		(instances
-			(project "CRSF-Multiswitch-ESP32-C3"
+			(project "RC-Multiswitch-ESP32-C3"
 				(path "/0f0fc713-9c7c-45b9-9629-0d42632ffdae"
 					(reference "#PWR01")
@@
 		)
 		(instances
-			(project "CRSF-Multiswitch-ESP32-C3"
+			(project "RC-Multiswitch-ESP32-C3"
 				(path "/0f0fc713-9c7c-45b9-9629-0d42632ffdae"
 					(reference "CN1")
@@
 		)
 		(instances
-			(project "CRSF-Multiswitch-ESP32-C3"
+			(project "RC-Multiswitch-ESP32-C3"
 				(path "/0f0fc713-9c7c-45b9-9629-0d42632ffdae"
 					(reference "R15")
@@
 		)
 		(instances
-			(project "CRSF-Multiswitch-ESP32-C3"
+			(project "RC-Multiswitch-ESP32-C3"
 				(path "/0f0fc713-9c7c-45b9-9629-0d42632ffdae"
 					(reference "LED6")
@@
 		)
 		(instances
-			(project "CRSF-Multiswitch-ESP32-C3"
+			(project "RC-Multiswitch-ESP32-C3"
 				(path "/0f0fc713-9c7c-45b9-9629-0d42632ffdae"
 					(reference "R11")
@@
 		)
 		(instances
-			(project "CRSF-Multiswitch-ESP32-C3"
+			(project "RC-Multiswitch-ESP32-C3"
 				(path "/0f0fc713-9c7c-45b9-9629-0d42632ffdae"
 					(reference "#PWR18")
@@
 		)
 		(instances
-			(project "CRSF-Multiswitch-ESP32-C3"
+			(project "RC-Multiswitch-ESP32-C3"
 				(path "/0f0fc713-9c7c-45b9-9629-0d42632ffdae"
 					(reference "#FLG08")
@@
 		)
 		(instances
-			(project "CRSF-Multiswitch-ESP32-C3"
+			(project "RC-Multiswitch-ESP32-C3"
 				(path "/0f0fc713-9c7c-45b9-9629-0d42632ffdae"
 					(reference "U1")
@@
 		)
 		(instances
-			(project "CRSF-Multiswitch-ESP32-C3"
+			(project "RC-Multiswitch-ESP32-C3"
 				(path "/0f0fc713-9c7c-45b9-9629-0d42632ffdae"
 					(reference "#PWR20")
@@
 		)
 		(instances
-			(project "CRSF-Multiswitch-ESP32-C3"
+			(project "RC-Multiswitch-ESP32-C3"
 				(path "/0f0fc713-9c7c-45b9-9629-0d42632ffdae"
 					(reference "#PWR22")
@@
 		)
 		(instances
-			(project "CRSF-Multiswitch-ESP32-C3"
+			(project "RC-Multiswitch-ESP32-C3"
 				(path "/0f0fc713-9c7c-45b9-9629-0d42632ffdae"
 					(reference "#PWR14")
@@
 		)
 		(instances
-			(project "CRSF-Multiswitch-ESP32-C3"
+			(project "RC-Multiswitch-ESP32-C3"
 				(path "/0f0fc713-9c7c-45b9-9629-0d42632ffdae"
 					(reference "LED1")
@@
 		)
 		(instances
-			(project "CRSF-Multiswitch-ESP32-C3"
+			(project "RC-Multiswitch-ESP32-C3"
 				(path "/0f0fc713-9c7c-45b9-9629-0d42632ffdae"
 					(reference "#PWR11")
@@
 		)
 		(instances
-			(project "CRSF-Multiswitch-ESP32-C3"
+			(project "RC-Multiswitch-ESP32-C3"
 				(path "/0f0fc713-9c7c-45b9-9629-0d42632ffdae"
 					(reference "#FLG05")
@@
 		)
 		(instances
-			(project "CRSF-Multiswitch-ESP32-C3"
+			(project "RC-Multiswitch-ESP32-C3"
 				(path "/0f0fc713-9c7c-45b9-9629-0d42632ffdae"
 					(reference "#PWR04")
@@
 		)
 		(instances
-			(project "CRSF-Multiswitch-ESP32-C3"
+			(project "RC-Multiswitch-ESP32-C3"
 				(path "/0f0fc713-9c7c-45b9-9629-0d42632ffdae"
 					(reference "#PWR16")
@@
 		)
 		(instances
-			(project "CRSF-Multiswitch-ESP32-C3"
+			(project "RC-Multiswitch-ESP32-C3"
 				(path "/0f0fc713-9c7c-45b9-9629-0d42632ffdae"
 					(reference "R4")
@@
 		)
 		(instances
-			(project "CRSF-Multiswitch-ESP32-C3"
+			(project "RC-Multiswitch-ESP32-C3"
 				(path "/0f0fc713-9c7c-45b9-9629-0d42632ffdae"
 					(reference "#PWR02")
@@
 		)
 		(instances
-			(project "CRSF-Multiswitch-ESP32-C3"
+			(project "RC-Multiswitch-ESP32-C3"
 				(path "/0f0fc713-9c7c-45b9-9629-0d42632ffdae"
 					(reference "LED2")
@@
 		)
 		(instances
-			(project "CRSF-Multiswitch-ESP32-C3"
+			(project "RC-Multiswitch-ESP32-C3"
 				(path "/0f0fc713-9c7c-45b9-9629-0d42632ffdae"
 					(reference "#PWR07")
@@
 		)
 		(instances
-			(project "CRSF-Multiswitch-ESP32-C3"
+			(project "RC-Multiswitch-ESP32-C3"
 				(path "/0f0fc713-9c7c-45b9-9629-0d42632ffdae"
 					(reference "R6")
@@
 		)
 		(instances
-			(project "CRSF-Multiswitch-ESP32-C3"
+			(project "RC-Multiswitch-ESP32-C3"
 				(path "/0f0fc713-9c7c-45b9-9629-0d42632ffdae"
 					(reference "#PWR21")
@@
 		)
 		(instances
-			(project "CRSF-Multiswitch-ESP32-C3"
+			(project "RC-Multiswitch-ESP32-C3"
 				(path "/0f0fc713-9c7c-45b9-9629-0d42632ffdae"
 					(reference "R9")
@@
 		)
 		(instances
-			(project "CRSF-Multiswitch-ESP32-C3"
+			(project "RC-Multiswitch-ESP32-C3"
 				(path "/0f0fc713-9c7c-45b9-9629-0d42632ffdae"
 					(reference "#PWR19")
@@
 		)
 		(instances
-			(project "CRSF-Multiswitch-ESP32-C3"
+			(project "RC-Multiswitch-ESP32-C3"
 				(path "/0f0fc713-9c7c-45b9-9629-0d42632ffdae"
 					(reference "#PWR17")
@@
 		)
 		(instances
-			(project "CRSF-Multiswitch-ESP32-C3"
+			(project "RC-Multiswitch-ESP32-C3"
 				(path "/0f0fc713-9c7c-45b9-9629-0d42632ffdae"
 					(reference "LED7")
@@
 		)
 		(instances
-			(project "CRSF-Multiswitch-ESP32-C3"
+			(project "RC-Multiswitch-ESP32-C3"
 				(path "/0f0fc713-9c7c-45b9-9629-0d42632ffdae"
 					(reference "#PWR12")
@@
 		)
 		(instances
-			(project "CRSF-Multiswitch-ESP32-C3"
+			(project "RC-Multiswitch-ESP32-C3"
 				(path "/0f0fc713-9c7c-45b9-9629-0d42632ffdae"
 					(reference "R13")
@@
 		)
 		(instances
-			(project "CRSF-Multiswitch-ESP32-C3"
+			(project "RC-Multiswitch-ESP32-C3"
 				(path "/0f0fc713-9c7c-45b9-9629-0d42632ffdae"
 					(reference "J5")
@@
 		)
 		(instances
-			(project "CRSF-Multiswitch-ESP32-C3"
+			(project "RC-Multiswitch-ESP32-C3"
 				(path "/0f0fc713-9c7c-45b9-9629-0d42632ffdae"
 					(reference "#PWR09")
@@
 		)
 		(instances
-			(project "CRSF-Multiswitch-ESP32-C3"
+			(project "RC-Multiswitch-ESP32-C3"
 				(path "/0f0fc713-9c7c-45b9-9629-0d42632ffdae"
 					(reference "R1")
@@
 		)
 		(instances
-			(project "CRSF-Multiswitch-ESP32-C3"
+			(project "RC-Multiswitch-ESP32-C3"
 				(path "/0f0fc713-9c7c-45b9-9629-0d42632ffdae"
 					(reference "R8")
@@
 		)
 		(instances
-			(project "CRSF-Multiswitch-ESP32-C3"
+			(project "RC-Multiswitch-ESP32-C3"
 				(path "/0f0fc713-9c7c-45b9-9629-0d42632ffdae"
 					(reference "R5")
@@
 		)
 		(instances
-			(project "CRSF-Multiswitch-ESP32-C3"
+			(project "RC-Multiswitch-ESP32-C3"
 				(path "/0f0fc713-9c7c-45b9-9629-0d42632ffdae"
 					(reference "U2")
@@
 		)
 		(instances
-			(project "CRSF-Multiswitch-ESP32-C3"
+			(project "RC-Multiswitch-ESP32-C3"
 				(path "/0f0fc713-9c7c-45b9-9629-0d42632ffdae"
 					(reference "R14")
@@
 		)
 		(instances
-			(project "CRSF-Multiswitch-ESP32-C3"
+			(project "RC-Multiswitch-ESP32-C3"
 				(path "/0f0fc713-9c7c-45b9-9629-0d42632ffdae"
 					(reference "R7")
@@
 		)
 		(instances
-			(project "CRSF-Multiswitch-ESP32-C3"
+			(project "RC-Multiswitch-ESP32-C3"
 				(path "/0f0fc713-9c7c-45b9-9629-0d42632ffdae"
 					(reference "#PWR10")
@@
 		)
 		(instances
-			(project "CRSF-Multiswitch-ESP32-C3"
+			(project "RC-Multiswitch-ESP32-C3"
 				(path "/0f0fc713-9c7c-45b9-9629-0d42632ffdae"
 					(reference "R16")
@@
 		)
 		(instances
-			(project "CRSF-Multiswitch-ESP32-C3"
+			(project "RC-Multiswitch-ESP32-C3"
 				(path "/0f0fc713-9c7c-45b9-9629-0d42632ffdae"
 					(reference "R12")
@@
 		)
 		(instances
-			(project "CRSF-Multiswitch-ESP32-C3"
+			(project "RC-Multiswitch-ESP32-C3"
 				(path "/0f0fc713-9c7c-45b9-9629-0d42632ffdae"
 					(reference "R2")
@@
 		)
 		(instances
-			(project "CRSF-Multiswitch-ESP32-C3"
+			(project "RC-Multiswitch-ESP32-C3"
 				(path "/0f0fc713-9c7c-45b9-9629-0d42632ffdae"
 					(reference "LED3")
@@
 		)
 		(instances
-			(project "CRSF-Multiswitch-ESP32-C3"
+			(project "RC-Multiswitch-ESP32-C3"
 				(path "/0f0fc713-9c7c-45b9-9629-0d42632ffdae"
 					(reference "CN2")
@@
 		)
 		(instances
-			(project "CRSF-Multiswitch-ESP32-C3"
+			(project "RC-Multiswitch-ESP32-C3"
 				(path "/0f0fc713-9c7c-45b9-9629-0d42632ffdae"
 					(reference "LED8")
@@
 		)
 		(instances
-			(project "CRSF-Multiswitch-ESP32-C3"
+			(project "RC-Multiswitch-ESP32-C3"
 				(path "/0f0fc713-9c7c-45b9-9629-0d42632ffdae"
 					(reference "R3")
@@
 		)
 		(instances
-			(project "CRSF-Multiswitch-ESP32-C3"
+			(project "RC-Multiswitch-ESP32-C3"
 				(path "/0f0fc713-9c7c-45b9-9629-0d42632ffdae"
 					(reference "J1")
@@
 		)
 		(instances
-			(project "CRSF-Multiswitch-ESP32-C3"
+			(project "RC-Multiswitch-ESP32-C3"
 				(path "/0f0fc713-9c7c-45b9-9629-0d42632ffdae"
 					(reference "#PWR03")
@@
 		)
 		(instances
-			(project "CRSF-Multiswitch-ESP32-C3"
+			(project "RC-Multiswitch-ESP32-C3"
 				(path "/0f0fc713-9c7c-45b9-9629-0d42632ffdae"
 					(reference "D1")
@@
 		)
 		(instances
-			(project "CRSF-Multiswitch-ESP32-C3"
+			(project "RC-Multiswitch-ESP32-C3"
 				(path "/0f0fc713-9c7c-45b9-9629-0d42632ffdae"
 					(reference "#PWR13")
@@
 		)
 		(instances
-			(project "CRSF-Multiswitch-ESP32-C3"
+			(project "RC-Multiswitch-ESP32-C3"
 				(path "/0f0fc713-9c7c-45b9-9629-0d42632ffdae"
 					(reference "R10")

Commit message: Lastversorgung CN2 auf 5-12 V, Widerstandswerte entfernt
- D1 TVS P6KE33A -> P6KE18A (Schaltplan, PCB, Aufdruck)
- Beschriftung CN2/VLOAD 12-24V -> 5-12V, Aufdruck 5V-24V -> 5V-12V
- R1-R16 ohne Wert: Anwender legt sie selbst aus, LED-Empfehlung steht auf der Platine
- Projektbeschreibung, Hardware-Beschreibung, README angepasst
- ULN2803A und ESP-Versorgung ueber CN1 bleiben unveraendert

Co-Authored-By: Claude Opus 5.5 (1M context) <noreply@anthropic.com>
Claude-Session: https://claude.ai/code/session_015ZTAHN4h1MhX6WfGWCfmx3
Parts:
- CN2: value 12V -> 5-12V
- D1: value P6KE33A -> P6KE18A
- R1, R10, R11, R12, R13, R14, R15, R16, R2, R3, R4, R5, R6, R7, R8, R9: value 150 -> R
Other:
- note added: "D1: TVS Anode GND, Kathode VLOAD (P6KE18A: ok bis 12V)"
- note added: "Last: 5-12V, max. 500mA je Kanal. ESP32 wird aus +5V von CN1 (BEC/Empfaenger) versorgt. Adresse per Firmware/Web-UI/Lua. Keine Pulldowns, keine UART-Vorwiderstaende. R1-R16: Werte legt der Anwender je LED bzw. Verbraucher selbst aus (siehe Projektbeschreibung)."
- note added: "Lastversorgung 5-12V (VLOAD)"
- note removed: "D1: TVS Anode GND, Kathode VLOAD (P6KE33A: ok bis 24V)"
- note removed: "Last: max. 24V / 500mA je Kanal. ESP32 wird aus +5V von CN1 (BEC/Empfaenger) versorgt. Adresse per Firmware/Web-UI/Lua. Keine Pulldowns, keine UART-Vorwiderstaende. R9-R16 und R1-R8: Standard 150R, je Verbraucher waehlen."
- note removed: "Lastversorgung 12-24V (VLOAD)"
Changed lines of the file:
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@@
 		)
 	)
-	(text "Last: max. 24V / 500mA je Kanal. ESP32 wird aus +5V von CN1 (BEC/Empfaenger) versorgt. Adresse per Firmware/Web-UI/Lua. Keine Pulldowns, keine UART-Vorwiderstaende. R9-R16 und R1-R8: Standard 150R, je Verbraucher waehlen."
+	(text "Last: 5-12V, max. 500mA je Kanal. ESP32 wird aus +5V von CN1 (BEC/Empfaenger) versorgt. Adresse per Firmware/Web-UI/Lua. Keine Pulldowns, keine UART-Vorwiderstaende. R1-R16: Werte legt der Anwender je LED bzw. Verbraucher selbst aus (siehe Projektbeschreibung)."
 		(exclude_from_sim no)
 		(at 15 21 0)
@@
 		)
 	)
-	(text "D1: TVS Anode GND, Kathode VLOAD (P6KE33A: ok bis 24V)"
+	(text "D1: TVS Anode GND, Kathode VLOAD (P6KE18A: ok bis 12V)"
 		(exclude_from_sim no)
 		(at 30 66 0)
@@
 		)
 	)
-	(text "Lastversorgung 12-24V (VLOAD)"
+	(text "Lastversorgung 5-12V (VLOAD)"
 		(exclude_from_sim no)
 		(at 15 40 0)
@@
 			)
 		)
-		(property "Value" "150"
+		(property "Value" "R"
 			(at 218.44 124.92 270)
 			(effects
@@
 			)
 		)
-		(property "Value" "150"
+		(property "Value" "R"
 			(at 218.44 94.44 270)
 			(effects
@@
 			)
 		)
-		(property "Value" "150"
+		(property "Value" "R"
 			(at 116.84 102.06 270)
 			(effects
@@
 			)
 		)
-		(property "Value" "150"
+		(property "Value" "R"
 			(at 116.84 117.3 270)
 			(effects
@@
 			)
 		)
-		(property "Value" "150"
+		(property "Value" "R"
 			(at 218.44 79.2 270)
 			(effects
@@
 			)
 		)
-		(property "Value" "150"
+		(property "Value" "R"
 			(at 218.44 109.68 270)
 			(effects
@@
 			)
 		)
-		(property "Value" "150"
+		(property "Value" "R"
 			(at 116.84 79.2 270)
 			(effects
@@
 			)
 		)
-		(property "Value" "150"
+		(property "Value" "R"
 			(at 116.84 132.54 270)
 			(effects
@@
 			)
 		)
-		(property "Value" "150"
+		(property "Value" "R"
 			(at 116.84 109.68 270)
 			(effects
@@
 			)
 		)
-		(property "Value" "150"
+		(property "Value" "R"
 			(at 218.44 117.3 270)
 			(effects
@@
 			)
 		)
-		(property "Value" "150"
+		(property "Value" "R"
 			(at 116.84 124.92 270)
 			(effects
@@
 			)
 		)
-		(property "Value" "150"
+		(property "Value" "R"
 			(at 218.44 132.54 270)
 			(effects
@@
 			)
 		)
-		(property "Value" "150"
+		(property "Value" "R"
 			(at 218.44 102.06 270)
 			(effects
@@
 			)
 		)
-		(property "Value" "150"
+		(property "Value" "R"
 			(at 116.84 86.82 270)
 			(effects
@@
 			)
 		)
-		(property "Value" "12V"
+		(property "Value" "5-12V"
 			(at 35.56 59.38 0)
 			(effects
@@
 			)
 		)
-		(property "Value" "150"
+		(property "Value" "R"
 			(at 116.84 94.44 270)
 			(effects
@@
 			)
 		)
-		(property "Value" "P6KE33A"
+		(property "Value" "P6KE18A"
 			(at 71.12 56.84 0)
 			(effects
@@
 			)
 		)
-		(property "Value" "150"
+		(property "Value" "R"
 			(at 218.44 86.82 270)
 			(effects
